File: KiCAD/TS100C.sch (KiCad schematic (older format))
At the start: 63 parts, among them J1 USB_C_Receptacle_USB2.0, J2 OLED_64x32, J3 A, J4 B, J5 DNP, P1 TC2030-CTX, Q1 SS8050, Q2 DMP3017SFG, SW1 key1, SW2 key2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

Commit message: Hook up SW1 to BOOT0 too
Parts:
- R24: renamed from J5; value DNP -> 2k3
- R5: value 2k37 -> 10k
- U3: symbol otter:STUSB4500 -> TS100C-rescue:STUSB4500-otter
- U7: symbol otter:SI8540 -> TS100C-rescue:SI8540-otter
Connections:
- net labels added: BOOT0
- wire segments 200 -> 205
- no-connect marks 7 -> 33
Changed lines of the file:
@@
 EESchema Schematic File Version 4
-LIBS:TS100C-cache
 EELAYER 30 0
 EELAYER END
@@
 $EndComp
 $Comp
-L power:+3V3 #PWR0102
-U 1 1 5A9AC22A
-P 5750 1100
-F 0 "#PWR0102" H 5750 950 50  0001 C CNN
-F 1 "+3V3" H 5765 1273 50  0000 C CNN
-F 2 "" H 5750 1100 50  0001 C CNN
-F 3 "" H 5750 1100 50  0001 C CNN
-	1    5750 1100
-	1    0    0    -1
-$EndComp
-$Comp
 L power:+3V3 #PWR0103
 U 1 1 5A9AC2BE
@@
 P 5750 1850
 F 0 "R5" H 5680 1804 50  0000 R CNN
-F 1 "2k37" H 5680 1895 50  0000 R CNN
+F 1 "10k" H 5680 1895 50  0000 R CNN
 F 2 "Resistor_SMD:R_0402_1005Metric" V 5680 1850 50  0001 C CNN
 F 3 "~" H 5750 1850 50  0001 C CNN
@@
 L power:VBUS #PWR?
 U 1 1 5BD81A2C
-P 2100 2250
+P 2100 2100
 AR Path="/588FA5F7/5BD81A2C" Ref="#PWR?"  Part="1"
 AR Path="/588FD270/5BD81A2C" Ref="#PWR?"  Part="1"
 AR Path="/5BD81A2C" Ref="#PWR0118"  Part="1"
-F 0 "#PWR0118" H 2100 2100 50  0001 C CNN
-F 1 "VBUS" H 2115 2423 50  0000 C CNN
-F 2 "" H 2100 2250 50  0001 C CNN
-F 3 "" H 2100 2250 50  0001 C CNN
-	1    2100 2250
+F 0 "#PWR0118" H 2100 1950 50  0001 C CNN
+F 1 "VBUS" H 2115 2273 50  0000 C CNN
+F 2 "" H 2100 2100 50  0001 C CNN
+F 3 "" H 2100 2100 50  0001 C CNN
+	1    2100 2100
 	1    0    0    -1
 $EndComp
@@
 	8350 2700 8050 2700
 Wire Wire Line
-	8050 2800 9150 2800
+	8050 2800 8750 2800
 Wire Wire Line
 	2300 5700 2150 5700
@@
 	11400 7450 11300 7450
 Wire Wire Line
-	2100 2250 1950 2250
-Wire Wire Line
 	1950 2750 1950 2850
 Wire Wire Line
@@
 	9250 7150 9100 7150
 $Comp
-L Device:R J5
+L Device:R R24
 U 1 1 5BE7685C
 P 5750 1350
-F 0 "J5" H 5680 1304 50  0000 R CNN
-F 1 "DNP" H 5680 1395 50  0000 R CNN
+F 0 "R24" H 5680 1304 50  0000 R CNN
+F 1 "2k3" H 5680 1395 50  0000 R CNN
 F 2 "Resistor_SMD:R_0402_1005Metric" V 5680 1350 50  0001 C CNN
 F 3 "~" H 5750 1350 50  0001 C CNN
@@
 Connection ~ 3500 7850
 $Comp
-L otter:STUSB4500 U3
+L TS100C-rescue:STUSB4500-otter U3
 U 1 1 5CE79B83
 P 4300 7900
@@
 Connection ~ 1350 3750
 $Comp
-L otter:SI8540 U7
+L TS100C-rescue:SI8540-otter U7
 U 1 1 5D0B5ED1
 P 13850 2200
@@
 Text GLabel 2150 2550 2    60   Input ~ 0
 CC2
+NoConn ~ 1950 3350
+NoConn ~ 1950 3450
+NoConn ~ 8050 4000
+NoConn ~ 8050 3500
+NoConn ~ 8050 3200
+NoConn ~ 8050 3100
+NoConn ~ 6750 1800
+NoConn ~ 6750 1900
+NoConn ~ 6750 2100
+NoConn ~ 6750 2200
+NoConn ~ 6750 2300
+NoConn ~ 6750 2500
+NoConn ~ 6750 2600
+NoConn ~ 6750 2700
+NoConn ~ 6750 2800
+NoConn ~ 6750 2900
+NoConn ~ 6750 3000
+NoConn ~ 6750 3300
+NoConn ~ 6750 3400
+NoConn ~ 6750 3800
+NoConn ~ 6750 3900
+NoConn ~ 6750 4000
+NoConn ~ 13950 7300
+NoConn ~ 13950 7000
+$Comp
+L power:PWR_FLAG #FLG0101
+U 1 1 5E16D266
+P 1550 3750
+F 0 "#FLG0101" H 1550 3825 50  0001 C CNN
+F 1 "PWR_FLAG" V 1550 3878 50  0000 L CNN
+F 2 "" H 1550 3750 50  0001 C CNN
+F 3 "~" H 1550 3750 50  0001 C CNN
+	1    1550 3750
+	0    1    1    0
+$EndComp
+Wire Wire Line
+	1550 3750 1350 3750
+$Comp
+L power:PWR_FLAG #FLG0102
+U 1 1 5E178BC3
+P 2200 2250
+F 0 "#FLG0102" H 2200 2325 50  0001 C CNN
+F 1 "PWR_FLAG" V 2200 2378 50  0000 L CNN
+F 2 "" H 2200 2250 50  0001 C CNN
+F 3 "~" H 2200 2250 50  0001 C CNN
+	1    2200 2250
+	0    1    1    0
+$EndComp
+Wire Wire Line
+	1950 2250 2100 2250
+Wire Wire Line
+	2100 2250 2100 2100
+Connection ~ 2100 2250
+Wire Wire Line
+	2100 2250 2200 2250
+NoConn ~ 8050 3400
+NoConn ~ 2150 5800
+Text GLabel 8750 2350 1    50   Input ~ 0
+BOOT0
+Wire Wire Line
+	8750 2350 8750 2800
+Connection ~ 8750 2800
+Wire Wire Line
+	8750 2800 9150 2800
+Text GLabel 5750 1100 1    50   Input ~ 0
+BOOT0
 $EndSCHEMATC
